File: schematics/javamon-v3.0.sch (EAGLE design)
At the start: 23 parts, among them IC1 ATmega328p, IC2 ESP-01, Q1 NTD4960N, U2 LD1086-3.3, X1 8MHz

Commit message: circuit redesign
Parts:
- removed X1: 8MHz, Crystals and Oscillators:RESONATOR-SMD_WIDE
Connections:
- removed net N$5: IC1.XTAL2/TOSC2, X1.3
- removed net N$6: IC1.XTAL1/TOSC1, X1.1
- net !B_UNIT: now also IC1.RXD; no longer IC1.ADC1
- net !B_ZERO: now also IC1.TXD; no longer IC1.ADC2
- net !ESP_RST: now also IC1.INT1; no longer IC1.ADC3
- net GND-D: no longer X1.2
- net LCD10: now also IC1.MISO; no longer IC1.RXD
- net LCD11: now also IC1.MOSI/OC2A; no longer IC1.SCK
- net LCD12: now also IC1.~SS/OC1B; no longer IC1.MISO
- net LCD13: now also IC1.OC1A; no longer IC1.MOSI/OC2A
- net LCD14: now also IC1.CLK0/ICP1; no longer IC1.~SS/OC1B
- net LCD15: now also IC1.T1/OC0B; no longer IC1.OC1A
- net LCD16: now also IC1.XCK/T0; no longer IC1.CLK0/ICP1
- net LCD5: no longer IC1.T1/OC0B
- net LCD6: no longer IC1.XCK/T0
- net LCD7: now also IC1.XTAL2/TOSC2; no longer IC1.INT1
- net LCD8: now also IC1.XTAL1/TOSC1; no longer IC1.INT0
- net LCD9: now also IC1.SCK; no longer IC1.TXD
- net S_PWR_CTL: now also IC1.INT0; no longer IC1.ADC0
Other:
- moved on the sheet: R2, R3
